Commit message: adjusted some values in the model

File: model/qb_legs.urdf.xacro (robot description, xacro)
@@ -17,4 +17,5 @@
 	<xacro:property name="torso_mass" value="2.7" />
 	<xacro:property name="foot_mass" value="0.75" />
+	<xacro:property name="pelvis_mass" value="0.3" />
 	<!-- isLeft parameter should be 1 for the left leg, -1 for the right leg -->
 	<xacro:macro name="qb_single_leg" params="parent name side isLeft high_joint mid_joint low_joint position orientation">
@@ -51,31 +52,42 @@
 			<insert_block name="origin" />
 			<parent link="${parent}" />
-			<child link="${name}_dummy_link" />
+			<child link="${name}_pelvis_link" />
 		</joint>
-		<link name="${name}_dummy_link"/>
+		<link name="${name}_pelvis_link">
+			<inertial>
+				<origin xyz="0 0 0" rpy="0 0 0" />
+				<mass value="${pelvis_mass}"/>
+				<inertia ixx="${pelvis_mass * cube_size * cube_size /9.0 * mm2_to_m2}" ixy="0.0" ixz="0.0" iyy="${pelvis_mass * legs_width * legs_width /9.0 * mm2_to_m2}" iyz="0.0" izz="${pelvis_mass * 20 * 20 /9.0 * mm2_to_m2}"/>
+			</inertial>
+			<visual>
+				<geometry>
+					<box size="${cube_size/scale_f} ${legs_width/scale_f} ${20/scale_f}"/>
+				</geometry>
+			</visual>
+		</link>
 		<!-- macro for each cube -->
 		<!-- torso -->
-		<xacro:qb_move parent="${name}_dummy_link" name="${name}_7" position="0 0 ${(flat_shaft/2.0+cube_size/2.0)/scale_f}" orientation="${- pi / 2} 0 0"/>
+		<xacro:qb_move parent="${name}_pelvis_link" name="${name}_7" position="0 0 ${(flat_shaft/2.0+cube_size/2.0)/scale_f}" orientation="${- pi / 2} 0 0"/>
 		<xacro:rotating_c_shaft parent="${name}_7" name="${name}_upper_shaft" position="0 0 0" orientation="${-pi / 2} 0 0"/>
 		<joint name="${name}_torso_joint" type="fixed">
 			<origin position="0 0 ${-(150-c_flange))/scale_f}" orientation="0 0 0"/>
 			<parent link="${name}_upper_shaft"/>
-			<child link="${name}_torso_box"/>
+			<child link="${name}_torso_link"/>
 		</joint>
-		<link name="${name}_torso_box">
+		<link name="${name}_torso_link">
 			<inertial>
 				<origin xyz="0 0 0" rpy="0 0 0" />
 				<mass value="${torso_mass}"/>
-				<inertia ixx="${torso_mass * 230 * 230 /9.0 * mm2_to_m2}" ixy="0.0" ixz="0.0" iyy="${torso_mass * 350 * 350 /9.0 * mm2_to_m2}" iyz="0.0" izz="${torso_mass * 100 * 100 /9.0 * mm2_to_m2}"/>
+				<inertia ixx="${torso_mass * 350 * 350 /9.0 * mm2_to_m2}" ixy="0.0" ixz="0.0" iyy="${torso_mass * 250 * 250 /9.0 * mm2_to_m2}" iyz="0.0" izz="${torso_mass * 100 * 100 /9.0 * mm2_to_m2}"/>
 			</inertial>
 			<visual>
 				<geometry>
-					<box size="${230/scale_f} ${350/scale_f} ${100/scale_f}"/>
+					<box size="${350/scale_f} ${250/scale_f} ${100/scale_f}"/>
 				</geometry>
 			</visual>
 		</link>
 		<!-- left leg -->
-		<xacro:qb_single_leg parent="${name}_dummy_link" name="${name}" side="left" isLeft="1" high_joint="3" mid_joint="2" low_joint="1" position="0 ${(legs_width-cube_size)/scale_f/2.0} ${-(flat_shaft/2.0+cube_size/2.0)/scale_f}" orientation="${-pi/2} 0 0"/>
-		<!-- <xacro:qb_move parent="${name}_dummy_link" name="${name}_3" position="0 ${(legs_width-cube_size)/scale_f/2.0} ${-(flat_shaft/2.0+cube_size/2.0)/scale_f}" orientation="${-pi/2} 0 0"/>
+		<xacro:qb_single_leg parent="${name}_pelvis_link" name="${name}" side="left" isLeft="1" high_joint="3" mid_joint="2" low_joint="1" position="0 ${(legs_width-cube_size)/scale_f/2.0} ${-(flat_shaft/2.0+cube_size/2.0)/scale_f}" orientation="${-pi/2} 0 0"/>
+		<!-- <xacro:qb_move parent="${name}_pelvis_link" name="${name}_3" position="0 ${(legs_width-cube_size)/scale_f/2.0} ${-(flat_shaft/2.0+cube_size/2.0)/scale_f}" orientation="${-pi/2} 0 0"/>
 		<xacro:rotating_c2_shaft parent="${name}_3" name="${name}_left_high_shaft" position="0 0 0" orientation="${pi/2} 0 0"/>
 		<xacro:qb_move parent="${name}_left_high_shaft" name="${name}_2" position="0 0 ${-extra_after_c2_flange/scale_f}" orientation="${-pi/2} 0 0"/>
@@ -98,8 +110,8 @@
 		</link> -->
 		<!-- right leg -->
-		<xacro:qb_single_leg parent="${name}_dummy_link" name="${name}" side="right" isLeft="-1" high_joint="4" mid_joint="5" low_joint="6" position="0 ${-(legs_width-cube_size)/scale_f/2.0} ${-(flat_shaft/2.0+cube_size/2.0)/scale_f}" orientation="${pi/2} 0 0"/>
+		<xacro:qb_single_leg parent="${name}_pelvis_link" name="${name}" side="right" isLeft="-1" high_joint="4" mid_joint="5" low_joint="6" position="0 ${-(legs_width-cube_size)/scale_f/2.0} ${-(flat_shaft/2.0+cube_size/2.0)/scale_f}" orientation="${pi/2} 0 0"/>
 		<!-- this is the same as the right leg, changing names and multiplying all roll angles by -1 -->
 		<!-- I'm keeping it separate for numbering convention -->
-		<!-- <xacro:qb_move parent="${name}_dummy_link" name="${name}_4" position="0 ${-(legs_width-cube_size)/scale_f/2.0} ${-(flat_shaft/2.0+cube_size/2.0)/scale_f}" orientation="${pi/2} 0 0"/>
+		<!-- <xacro:qb_move parent="${name}_pelvis_link" name="${name}_4" position="0 ${-(legs_width-cube_size)/scale_f/2.0} ${-(flat_shaft/2.0+cube_size/2.0)/scale_f}" orientation="${pi/2} 0 0"/>
 		<xacro:rotating_c2_shaft parent="${name}_4" name="${name}_right_high_shaft" position="0 0 0" orientation="${-pi/2} 0 0"/>
 		<xacro:qb_move parent="${name}_right_high_shaft" name="${name}_5" position="0 0 ${-extra_after_c2_flange/scale_f}" orientation="${pi/2} 0 0"/>

File: model/qb_utility_models.urdf.xacro (robot description, xacro)
@@ -5,6 +5,6 @@
 	<xacro:property name="c2_flange" value="120" />
 	<xacro:property name="flange_mass" value="0.1" />
-	<xacro:property name="c_flange_com_z" value="15" />
-	<xacro:property name="c2_flange_com_z" value="44" />
+	<xacro:property name="c_flange_com_z" value="48" />
+	<xacro:property name="c2_flange_com_z" value="72" />
 	<xacro:property name="mp_cube_mass" value="0.25" />
 	<!-- a macro for non-actuated qb cubes -->
@@ -77,5 +77,5 @@
 		<link name="${name}_link">
 			<inertial>
-				<origin xyz="0 0 ${-(cube_size/2.0+c_flange_com_z)/scale_f}" rpy="0 0 0" />
+				<origin xyz="0 0 ${-(c_flange_com_z)/scale_f}" rpy="0 0 0" />
 				<mass value="${flange_mass}"/>
 				<inertia ixx="${flange_mass * cube_size * cube_size /9.0 * mm2_to_m2}" ixy="0.0" ixz="0.0" iyy="${flange_mass * cube_size * cube_size /9.0 * mm2_to_m2}" iyz="0.0" izz="${flange_mass * cube_size * cube_size /9.0 * mm2_to_m2}"/>
@@ -110,5 +110,5 @@
 		<link name="${name}_link">
 			<inertial>
-				<origin xyz="0 0 ${-(cube_size/2.0+c_flange_com_z)/scale_f}" rpy="0 0 0" />
+				<origin xyz="0 0 ${(-c_flange+c_flange_com_z)/scale_f}" rpy="0 0 0" />
 				<mass value="${flange_mass}"/>
 				<inertia ixx="${flange_mass * cube_size * cube_size /9.0 * mm2_to_m2}" ixy="0.0" ixz="0.0" iyy="${flange_mass * cube_size * cube_size /9.0 * mm2_to_m2}" iyz="0.0" izz="${flange_mass * cube_size * cube_size /9.0 * mm2_to_m2}"/>
@@ -142,5 +142,5 @@
 		<link name="${name}_link">
 			<inertial>
-				<origin xyz="0 0 ${-(cube_size/2.0+c2_flange_com_z)/scale_f}" rpy="0 0 0" />
+				<origin xyz="0 0 ${-(c2_flange_com_z)/scale_f}" rpy="0 0 0" />
 				<mass value="${flange_mass}"/>
 				<inertia ixx="${flange_mass * cube_size * cube_size /9.0 * mm2_to_m2}" ixy="0.0" ixz="0.0" iyy="${flange_mass * cube_size * cube_size /9.0 * mm2_to_m2}" iyz="0.0" izz="${flange_mass * cube_size * cube_size /9.0 * mm2_to_m2}"/>

Commit message: removed useless comments in legs model file

File: model/qb_legs.urdf.xacro (robot description, xacro)
@@ -2,5 +2,4 @@
 <robot xmlns:xacro="http://www.ros.org/wiki/xacro">
 	<!-- we need the definition of the qb_move unit -->
-	<!-- <xacro:include filename="$(find qbmove_description)/model/qb_move.urdf.xacro" /> -->
 	<xacro:include filename="$(find qb_legs)/model/qb_utility_models.urdf.xacro" />
 	<xacro:property name="pi" value="3.1415926535897931" />
@@ -48,5 +47,5 @@
 	<xacro:macro name="qb_legs" params="parent name *origin">
 		<!-- macro for the robot -->
-		<!-- dummy link -->
+		<!-- pelvis link, attached to the external link -->
 		<joint name="${name}_dummy_joint" type="fixed" >
 			<insert_block name="origin" />
@@ -66,5 +65,4 @@
 			</visual>
 		</link>
-		<!-- macro for each cube -->
 		<!-- torso -->
 		<xacro:qb_move parent="${name}_pelvis_link" name="${name}_7" position="0 0 ${(flat_shaft/2.0+cube_size/2.0)/scale_f}" orientation="${- pi / 2} 0 0"/>
@@ -89,67 +87,6 @@
 		<!-- left leg -->
 		<xacro:qb_single_leg parent="${name}_pelvis_link" name="${name}" side="left" isLeft="1" high_joint="3" mid_joint="2" low_joint="1" position="0 ${(legs_width-cube_size)/scale_f/2.0} ${-(flat_shaft/2.0+cube_size/2.0)/scale_f}" orientation="${-pi/2} 0 0"/>
-		<!-- <xacro:qb_move parent="${name}_pelvis_link" name="${name}_3" position="0 ${(legs_width-cube_size)/scale_f/2.0} ${-(flat_shaft/2.0+cube_size/2.0)/scale_f}" orientation="${-pi/2} 0 0"/>
-		<xacro:rotating_c2_shaft parent="${name}_3" name="${name}_left_high_shaft" position="0 0 0" orientation="${pi/2} 0 0"/>
-		<xacro:qb_move parent="${name}_left_high_shaft" name="${name}_2" position="0 0 ${-extra_after_c2_flange/scale_f}" orientation="${-pi/2} 0 0"/>
-		<xacro:rotating_c_shaft parent="${name}_2" name="${name}_left_mid_shaft" position="0 0 0" orientation="${pi/2} 0 0"/>
-		<xacro:qb_empty parent="${name}_left_mid_shaft" name="${name}_left_empty" position="0 0 0" orientation="${-pi/2} 0 0"/>
-		<xacro:fixed_c_shaft parent="${name}_left_empty" name="${name}_left_low_shaft" position="0 0 0" orientation="${pi/2} 0 0"/>
-		<xacro:qb_move_reverse parent="${name}_left_low_shaft" name="${name}_1" position="0 0 ${-extra_after_c2_flange/scale_f}" orientation="${-pi/2} 0 0"/>
-		<joint name="${name}_left_foot_joint" type="fixed">
-			<origin xyz="0 ${foot_height/scale_f} 0" rpy="${pi/2} 0 0"/>
-			<parent link="${name}_1"/>
-			<child link="${name}_left_foot"/>
-		</joint>
-		<link name="${name}_left_foot">
-			<visual>
-				<origin xyz="0 0 ${foot_thickness/scale_f/2.0}" rpy="0 0 0"/>
-				<geometry>
-					<box size="${140/scale_f} ${cube_size/scale_f} ${foot_thickness/scale_f}"/>
-				</geometry>
-			</visual>
-		</link> -->
 		<!-- right leg -->
 		<xacro:qb_single_leg parent="${name}_pelvis_link" name="${name}" side="right" isLeft="-1" high_joint="4" mid_joint="5" low_joint="6" position="0 ${-(legs_width-cube_size)/scale_f/2.0} ${-(flat_shaft/2.0+cube_size/2.0)/scale_f}" orientation="${pi/2} 0 0"/>
-		<!-- this is the same as the right leg, changing names and multiplying all roll angles by -1 -->
-		<!-- I'm keeping it separate for numbering convention -->
-		<!-- <xacro:qb_move parent="${name}_pelvis_link" name="${name}_4" position="0 ${-(legs_width-cube_size)/scale_f/2.0} ${-(flat_shaft/2.0+cube_size/2.0)/scale_f}" orientation="${pi/2} 0 0"/>
-		<xacro:rotating_c2_shaft parent="${name}_4" name="${name}_right_high_shaft" position="0 0 0" orientation="${-pi/2} 0 0"/>
-		<xacro:qb_move parent="${name}_right_high_shaft" name="${name}_5" position="0 0 ${-extra_after_c2_flange/scale_f}" orientation="${pi/2} 0 0"/>
-		<xacro:rotating_c_shaft parent="${name}_5" name="${name}_right_mid_shaft" position="0 0 0" orientation="${-pi/2} 0 0"/>
-		<xacro:qb_empty parent="${name}_right_mid_shaft" name="${name}_right_empty" position="0 0 0" orientation="${pi/2} 0 0"/>
-		<xacro:fixed_c_shaft parent="${name}_right_empty" name="${name}_right_low_shaft" position="0 0 0" orientation="${-pi/2} 0 0"/>
-		<xacro:qb_move_reverse parent="${name}_right_low_shaft" name="${name}_6" position="0 0 ${-extra_after_c2_flange/scale_f}" orientation="${pi/2} 0 0"/>
-		<joint name="${name}_right_foot_joint" type="fixed">
-			<origin xyz="0 ${-foot_height/scale_f} 0" rpy="${-pi/2} 0 0"/>
-			<parent link="${name}_6"/>
-			<child link="${name}_right_foot"/>
-		</joint>
-		<link name="${name}_right_foot">
-			<visual>
-				<origin xyz="0 0 ${foot_thickness/scale_f/2.0}" rpy="0 0 0"/>
-				<geometry>
-					<box size="${140/scale_f} ${cube_size/scale_f} ${foot_thickness/scale_f}"/>
-				</geometry>
-			</visual>
-		</link> -->
-<!-- 		<xacro:qb_empty parent="${name}_upper_shaft" name="${name}_empty">
-			<origin position="0 0 0" orientation="0 0 0"/>
-		</xacro:qb_empty> -->
-			<!-- <origin position="0 0 ${one_flange/scale_f}" orientation="0 0 0"/> -->
-		<!-- if the fixed joint is a problem while planning, comment the following one -->
-		<!-- <xacro:qb_move parent="${name}_1" name="${name}_1bis" position="0 0 ${one_flange/scale_f}" orientation="0 ${pi / 2} 0" />
-		<xacro:qb_move parent="${name}_1" name="${name}_2" position="0 0 ${one_flange/scale_f+two_flanges/scale_f}" orientation="0 0 0" /> -->
-		<!-- right arm -->
-		<!-- <xacro:qb_move parent="${name}_1" name="${name}_20" position="0 ${- two_flanges/scale_f} ${one_flange/scale_f+two_flanges/scale_f}" orientation="0 ${- pi / 2} ${pi / 2}" />
-		<xacro:qb_move parent="${name}_20" name="${name}_21" position="0 0 ${one_flange/scale_f}" orientation="${pi / 2} 0 0" />
-		<xacro:qb_move parent="${name}_21" name="${name}_22" position="${- c_flange/scale_f} 0 0" orientation="0 ${- pi / 2} 0" />
-		<xacro:qb_move parent="${name}_22" name="${name}_23" position="0 0 ${one_flange/scale_f}" orientation="${pi / 2} 0 0" />
-		<xacro:qb_move parent="${name}_23" name="${name}_24" position="0 ${c_flange/scale_f} 0" orientation="0 0 0" /> -->
-		<!-- left arm -->
-		<!-- <xacro:qb_move parent="${name}_1" name="${name}_10" position="0 ${two_flanges/scale_f} ${one_flange/scale_f+two_flanges/scale_f}" orientation="0 ${- pi / 2} ${- pi / 2}" />
-		<xacro:qb_move parent="${name}_10" name="${name}_11" position="0 0 ${one_flange/scale_f}" orientation="${- pi / 2} 0 0" />
-		<xacro:qb_move parent="${name}_11" name="${name}_12" position="${- c_flange/scale_f} 0 0" orientation="0 ${- pi / 2} 0" />
-		<xacro:qb_move parent="${name}_12" name="${name}_13" position="0 0 ${one_flange/scale_f}" orientation="${pi / 2} 0 0" />
-		<xacro:qb_move parent="${name}_13" name="${name}_14" position="0 ${c_flange/scale_f} 0" orientation="${pi} 0 0" /> -->
 	</xacro:macro>
 </robot>

Commit message: approximated inertia values to full, uniform cuboids

File: model/qb_legs.urdf.xacro (robot description, xacro)
@@ -4,7 +4,4 @@
 	<xacro:include filename="$(find qb_legs)/model/qb_utility_models.urdf.xacro" />
 	<xacro:property name="pi" value="3.1415926535897931" />
-	<xacro:property name="one_flange" value="78" />
-	<xacro:property name="two_flanges" value="85" />
-	<xacro:property name="c_flange" value="90" />
 	<xacro:property name="flat_shaft" value="44" /> <!-- (110-66) -->
 	<xacro:property name="scale_f" value="1000" />
@@ -14,4 +11,6 @@
 	<xacro:property name="foot_com_height" value="24" />
 	<xacro:property name="foot_thickness" value="10" />
+	<xacro:property name="foot_length" value="140" />
+	<xacro:property name="pelvis_thickness" value="20" />
 	<xacro:property name="torso_mass" value="2.7" />
 	<xacro:property name="foot_mass" value="0.75" />
@@ -35,10 +34,10 @@
 				<origin xyz="0 0 ${foot_com_height/scale_f}" rpy="0 0 0" />
 				<mass value="${foot_mass}"/>
-				<inertia ixx="${foot_mass * 140 * 140 /9.0 * mm2_to_m2}" ixy="0.0" ixz="0.0" iyy="${foot_mass * cube_size * cube_size /9.0 * mm2_to_m2}" iyz="0.0" izz="${foot_mass * foot_thickness * foot_thickness /9.0 * mm2_to_m2}"/>
+				<inertia ixx="${foot_mass * (cube_size * cube_size + foot_thickness * foot_thickness) / 12.0 * mm2_to_m2}" ixy="0.0" ixz="0.0" iyy="${foot_mass * (foot_length * foot_length + foot_thickness * foot_thickness) / 12.0 * mm2_to_m2}" iyz="0.0" izz="${foot_mass * (foot_length * foot_length + cube_size * cube_size) / 12.0 * mm2_to_m2}"/>
 			</inertial>
 			<visual>
 				<origin xyz="0 0 ${foot_thickness/scale_f/2.0}" rpy="0 0 0"/>
 				<geometry>
-					<box size="${140/scale_f} ${cube_size/scale_f} ${foot_thickness/scale_f}"/>
+					<box size="${foot_length/scale_f} ${cube_size/scale_f} ${foot_thickness/scale_f}"/>
 				</geometry>
 			</visual>
@@ -57,9 +56,9 @@
 				<origin xyz="0 0 0" rpy="0 0 0" />
 				<mass value="${pelvis_mass}"/>
-				<inertia ixx="${pelvis_mass * cube_size * cube_size /9.0 * mm2_to_m2}" ixy="0.0" ixz="0.0" iyy="${pelvis_mass * legs_width * legs_width /9.0 * mm2_to_m2}" iyz="0.0" izz="${pelvis_mass * 20 * 20 /9.0 * mm2_to_m2}"/>
+				<inertia ixx="${pelvis_mass * (legs_width * legs_width + pelvis_thickness * pelvis_thickness) / 12.0 * mm2_to_m2}" ixy="0.0" ixz="0.0" iyy="${pelvis_mass * (cube_size * cube_size + pelvis_thickness * pelvis_thickness) / 12.0 * mm2_to_m2}" iyz="0.0" izz="${pelvis_mass * (cube_size * cube_size + legs_width * legs_width) / 12.0 * mm2_to_m2}"/>
 			</inertial>
 			<visual>
 				<geometry>
-					<box size="${cube_size/scale_f} ${legs_width/scale_f} ${20/scale_f}"/>
+					<box size="${cube_size/scale_f} ${legs_width/scale_f} ${pelvis_thickness/scale_f}"/>
 				</geometry>
 			</visual>
@@ -77,5 +76,5 @@
 				<origin xyz="0 0 0" rpy="0 0 0" />
 				<mass value="${torso_mass}"/>
-				<inertia ixx="${torso_mass * 350 * 350 /9.0 * mm2_to_m2}" ixy="0.0" ixz="0.0" iyy="${torso_mass * 250 * 250 /9.0 * mm2_to_m2}" iyz="0.0" izz="${torso_mass * 100 * 100 /9.0 * mm2_to_m2}"/>
+				<inertia ixx="${torso_mass * (250 * 250 + 100 * 100) / 12.0 * mm2_to_m2}" ixy="0.0" ixz="0.0" iyy="${torso_mass * (350 * 350 + 100 * 100) / 12.0 * mm2_to_m2}" iyz="0.0" izz="${torso_mass * (350 * 350 + 250 * 250) / 12.0 * mm2_to_m2}"/>
 			</inertial>
 			<visual>

File: model/qb_utility_models.urdf.xacro (robot description, xacro)
@@ -49,7 +49,8 @@
 		<link name="${name}">
 			<inertial>
+				<!-- inertia of a full, uniform cube -->
 				<origin xyz="0 0 0" rpy="0 0 0" />
 				<mass value="${mp_cube_mass}"/>
-				<inertia ixx="${mp_cube_mass * cube_size * cube_size /9.0 * mm2_to_m2}" ixy="0.0" ixz="0.0" iyy="${mp_cube_mass * cube_size * cube_size /9.0 * mm2_to_m2}" iyz="0.0" izz="${mp_cube_mass * cube_size * cube_size /9.0 * mm2_to_m2}"/>
+				<inertia ixx="${mp_cube_mass * cube_size * cube_size / 6.0 * mm2_to_m2}" ixy="0.0" ixz="0.0" iyy="${mp_cube_mass * cube_size * cube_size / 6.0 * mm2_to_m2}" iyz="0.0" izz="${mp_cube_mass * cube_size * cube_size / 6.0 * mm2_to_m2}"/>
 			</inertial>
 			<visual>
